File: eagle/welder_pcb.sch (EAGLE design)
At the start: 12 parts, among them IC2 7805TV, Q1 16MHz

Commit message: Add Relay Pins
Parts:
- added RELAY: (no value), pinhead:PINHD-1X3
Connections:
- new net OC1B: ATMEGA328P.16, RELAY.3
- net +5V: now also RELAY.2
- net GND: now also RELAY.1
Changed lines of the file:
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@@
 <part name="TRIM" library="pinhead" library_urn="urn:adsk.eagle:library:325" deviceset="PINHD-1X3" device="" package3d_urn="urn:adsk.eagle:package:22458/2"/>
 <part name="LCD" library="pinhead" library_urn="urn:adsk.eagle:library:325" deviceset="PINHD-1X3" device="" package3d_urn="urn:adsk.eagle:package:22458/2"/>
+<part name="RELAY" library="pinhead" library_urn="urn:adsk.eagle:library:325" deviceset="PINHD-1X3" device="" package3d_urn="urn:adsk.eagle:package:22458/2"/>
 </parts>
 <sheets>
@@
 <instance part="TRIM" gate="A" x="162.56" y="35.56"/>
 <instance part="LCD" gate="A" x="195.58" y="35.56"/>
+<instance part="RELAY" gate="A" x="127" y="83.82"/>
 </instances>
 <busses>
@@
 <label x="185.42" y="35.56" size="1.016" layer="95" rot="R180" xref="yes"/>
 </segment>
+<segment>
+<pinref part="RELAY" gate="A" pin="1"/>
+<wire x1="124.46" y1="86.36" x2="114.3" y2="86.36" width="0.1524" layer="91"/>
+<label x="114.3" y="86.36" size="1.016" layer="95" rot="R180" xref="yes"/>
+</segment>
 </net>
 <net name="N$1" class="0">
@@
 <label x="185.42" y="38.1" size="1.016" layer="95" rot="R180" xref="yes"/>
 </segment>
+<segment>
+<pinref part="RELAY" gate="A" pin="2"/>
+<wire x1="124.46" y1="83.82" x2="114.3" y2="83.82" width="0.1524" layer="91"/>
+<label x="114.3" y="83.82" size="1.016" layer="95" rot="R180" xref="yes"/>
+</segment>
 </net>
 <net name="RESET" class="0">
@@
 </segment>
 </net>
+<net name="OC1B" class="0">
+<segment>
+<pinref part="ATMEGA328P" gate="G$1" pin="16"/>
+<wire x1="50.8" y1="20.32" x2="53.34" y2="20.32" width="0.1524" layer="91"/>
+<label x="53.34" y="20.32" size="1.016" layer="95" xref="yes"/>
+</segment>
+<segment>
+<pinref part="RELAY" gate="A" pin="3"/>
+<wire x1="124.46" y1="81.28" x2="114.3" y2="81.28" width="0.1524" layer="91"/>
+<label x="114.3" y="81.28" size="1.016" layer="95" rot="R180" xref="yes"/>
+</segment>
+</net>
